File: ThreeMan_HW.kicad_pcb (KiCad board)
At the start: 2 copper layers, 5 parts, among them J1 USB4135-GF-A, U1 MCP73831T-2ACI/OT

Commit message: Finished initial draft of A1 schematic and imported it to PCB
Parts:
- removed G***: LOGO, Logo:Zkylark_10x8mm
- added C3: 100u, Capacitor_SMD:C_0603_HS, F.Cu at (89.5, 81.6)
- added C4: 100u, Capacitor_SMD:C_0603_HS, F.Cu at (89.5, 84.1)
- added C5: 100u, Capacitor_SMD:C_0603_HS, F.Cu at (89.5, 86.6)
- added C6: 100u, Capacitor_SMD:C_0603_HS, F.Cu at (89.5, 89.1)
- added C7: 100u, Capacitor_SMD:C_0603_HS, F.Cu at (89.5, 91.6)
- added C8: 100u, Capacitor_SMD:C_0603_HS, F.Cu at (89.5, 94.1)
- added C9: 100u, Capacitor_SMD:C_0603_HS, F.Cu at (89.5, 96.6)
- added D1: SMAJ5.0A, Diode_SMD:DO-214AC, F.Cu at (109.1, 113.9)
- added D10: Colour, LED_SMD:LED_0603_HS, F.Cu at (93.8, 94.1)
- added D11: Colour, LED_SMD:LED_0603_HS, F.Cu at (93.8, 96.6)
- added D12: Colour, LED_SMD:LED_0603_HS, F.Cu at (93.8, 99.1)
- added D13: Colour, LED_SMD:LED_0603_HS, F.Cu at (98.2, 76.5)
- added D14: Colour, LED_SMD:LED_0603_HS, F.Cu at (98.2, 79.0)
- added D15: Colour, LED_SMD:LED_0603_HS, F.Cu at (98.2, 81.6)
- added D16: Colour, LED_SMD:LED_0603_HS, F.Cu at (98.2, 84.1)
- added D17: Colour, LED_SMD:LED_0603_HS, F.Cu at (98.2, 86.6)
- added D2: Red, LED_SMD:LED_0603_HS, F.Cu at (89.5, 99.1)
- added D3: Green, LED_SMD:LED_0603_HS, F.Cu at (93.8, 76.5)
- added D4: Colour, LED_SMD:LED_0603_HS, F.Cu at (93.8, 79.0)
- added D5: Colour, LED_SMD:LED_0603_HS, F.Cu at (93.8, 81.6)
- added D6: Colour, LED_SMD:LED_0603_HS, F.Cu at (93.8, 84.1)
- added D7: Colour, LED_SMD:LED_0603_HS, F.Cu at (93.8, 86.6)
- added D8: Colour, LED_SMD:LED_0603_HS, F.Cu at (93.8, 89.1)
- added D9: Colour, LED_SMD:LED_0603_HS, F.Cu at (93.8, 91.6)
- added J2: JST-PH-2mm, Connector_JST:JST_PH_S2B-PH-SM4-TB_1x02-1MP_P2.00mm_Horizontal, F.Cu at (110.1, 106.0)
- added J3: TC2030_ICSP, Connector:Tag-Connect_TC2030-IDC-FP_2x03_P1.27mm_Vertical, F.Cu at (120.0, 105.2)
- added R1: 5k1, Resistor_SMD:R_0603_HS, F.Cu at (98.2, 89.1)
- added R10: 0R, Resistor_SMD:R_0603_HS, F.Cu at (102.5, 86.6)
- added R11: 0R, Resistor_SMD:R_0603_HS, F.Cu at (102.5, 89.1)
- added R12: 0R, Resistor_SMD:R_0603_HS, F.Cu at (102.5, 91.6)
- added R13: 0R, Resistor_SMD:R_0603_HS, F.Cu at (102.5, 94.1)
- added R14: 0R, Resistor_SMD:R_0603_HS, F.Cu at (102.5, 96.6)
- added R15: 0R, Resistor_SMD:R_0603_HS, F.Cu at (102.5, 99.1)
- added R16: 0R, Resistor_SMD:R_0603_HS, F.Cu at (106.9, 76.5)
- added R17: 0R, Resistor_SMD:R_0603_HS, F.Cu at (106.9, 79.0)
- added R18: 0R, Resistor_SMD:R_0603_HS, F.Cu at (106.9, 81.6)
- added R19: 0R, Resistor_SMD:R_0603_HS, F.Cu at (106.9, 84.1)
- added R2: 5k1, Resistor_SMD:R_0603_HS, F.Cu at (98.2, 91.6)
- added R20: 0R, Resistor_SMD:R_0603_HS, F.Cu at (106.9, 86.6)
- added R21: 0R, Resistor_SMD:R_0603_HS, F.Cu at (106.9, 89.1)
- added R22: 120R, Resistor_SMD:R_0603_HS, F.Cu at (106.9, 91.6)
- added R23: 120R, Resistor_SMD:R_0603_HS, F.Cu at (106.9, 94.1)
- added R24: 120R, Resistor_SMD:R_0603_HS, F.Cu at (106.9, 96.6)
- added R25: 120R, Resistor_SMD:R_0603_HS, F.Cu at (106.9, 99.1)
- added R26: 120R, Resistor_SMD:R_0603_HS, F.Cu at (111.2, 76.5)
- added R27: 120R, Resistor_SMD:R_0603_HS, F.Cu at (111.2, 79.0)
- added R28: 120R, Resistor_SMD:R_0603_HS, F.Cu at (111.2, 81.6)
- added R29: 120R, Resistor_SMD:R_0603_HS, F.Cu at (111.2, 84.1)
- added R3: R, Resistor_SMD:R_0603_HS, F.Cu at (98.2, 94.1)
- added R30: 120R, Resistor_SMD:R_0603_HS, F.Cu at (111.2, 86.6)
- added R31: 120R, Resistor_SMD:R_0603_HS, F.Cu at (111.2, 89.1)
- added R32: 120R, Resistor_SMD:R_0603_HS, F.Cu at (111.2, 91.6)
- added R33: 120R, Resistor_SMD:R_0603_HS, F.Cu at (111.2, 94.1)
- added R34: 120R, Resistor_SMD:R_0603_HS, F.Cu at (111.2, 96.6)
- added R35: 120R, Resistor_SMD:R_0603_HS, F.Cu at (111.2, 99.1)
- added R4: R, Resistor_SMD:R_0603_HS, F.Cu at (98.2, 96.6)
- added R5: 2k, Resistor_SMD:R_0603_HS, F.Cu at (98.2, 99.1)
- added R6: 0R, Resistor_SMD:R_0603_HS, F.Cu at (102.5, 76.5)
- added R7: 10k, Resistor_SMD:R_0603_HS, F.Cu at (102.5, 79.0)
- added R8: 0R, Resistor_SMD:R_0603_HS, F.Cu at (102.5, 81.6)
- added R9: 0R, Resistor_SMD:R_0603_HS, F.Cu at (102.5, 84.1)
- added SW1: Off-Mom, Switch_Button_SMD:SW_SPST_PTS645, F.Cu at (119.0, 87.5)
- added SW2: SW_SPDT_312, Switch_Slide_SMD:CSS-1210TB, F.Cu at (115.6, 77.0)
- added U2: 74HC595, Package_SO:TSSOP-16_4.4x5mm_P0.65mm, F.Cu at (119.6, 113.2)
- added U3: ATTINY85-20SUR, Package_SO:SOIC-8_5.3x5.3mm_P1.27mm, F.Cu at (118.7, 94.9)
- added U4: TPS7A20, Package_TO_SOT_SMD:SOT-23-5, F.Cu at (89.9, 114.3)
- added U5: ULQ2003D, Package_SO:SOIC-16-N_3.8x9.8mm_P1.27mm, F.Cu at (91.7, 106.2)
- added U6: ULQ2003D, Package_SO:SOIC-16-N_3.8x9.8mm_P1.27mm, F.Cu at (100.6, 106.2)
- C1: value xF -> 4u7; footprint Capacitor_SMD:C_0402 -> Capacitor_SMD:C_0603_HS
- C2: value xF -> 4u7; footprint Capacitor_SMD:C_0603_HandSolder -> Capacitor_SMD:C_0603_HS
- moved C2 54.4 mm to (89.5, 79.0)
- moved C1 53.9 mm to (89.5, 76.5), turned to 0 degrees
Connections:
- net Net-(J1-VBUS-PadA9) renamed /V_{USB}
- C1 pad 1: unconnected-(C1-Pad1) -> /V_{USB-filt}
- C1 pad 2: unconnected-(C1-Pad2) -> GND
- C2 pad 1: unconnected-(C2-Pad1) -> /V_{BAT}
- C2 pad 2: unconnected-(C2-Pad2) -> GND
- J1 pad A12: Net-(J1-GND-PadA12) -> GND
- J1 pad B12: Net-(J1-GND-PadA12) -> GND
- U1 pad 1: unconnected-(U1-STAT-Pad1) -> Net-(D2-K)
- U1 pad 2: unconnected-(U1-V_{SS}-Pad2) -> GND
- U1 pad 3: unconnected-(U1-V_{BAT}-Pad3) -> /V_{BAT}
- U1 pad 4: unconnected-(U1-V_{DD}-Pad4) -> /V_{USB-filt}
- U1 pad 5: unconnected-(U1-PROG-Pad5) -> Net-(U1-PROG)

Commit message: Completed layout
Parts:
- added H1: M3, MountingHole:MountingHole_3.2mm_M3_Pad, F.Cu at (118.5, 63.5)
- added H2: M3, MountingHole:MountingHole_3.2mm_M3_Pad, F.Cu at (191.5, 63.5)
- added H3: M3, MountingHole:MountingHole_3.2mm_M3_Pad, F.Cu at (118.5, 96.5)
- added H4: M3, MountingHole:MountingHole_3.2mm_M3_Pad, F.Cu at (191.5, 96.5)
- C3, C4, C5, C6, C7, C8, C9: value 100u -> 100n
- D11, D12, D13, D14, D15, D16, D17: value Colour -> Red
- D21: renamed from D4; value Colour -> Red
- D22: renamed from D5; value Colour -> Red
- D23: renamed from D6; value Colour -> Red
- D24: renamed from D7; value Colour -> Red
- D25: renamed from D8; value Colour -> Red
- D26: renamed from D9; value Colour -> Red
- D27: renamed from D10; value Colour -> Red
- R3, R4: value R -> 590R
- SW1: value Off-Mom -> SW_Push; footprint Switch_Button_SMD:SW_SPST_PTS645 -> Switch_Button_SMD:SW_SPST_TS04-66-95-BK-160-SMT
- moved D25 95.5 mm to (186.0, 64.0), turned to 180 degrees
- moved D27 95.4 mm to (186.0, 69.5), turned to 180 degrees
- moved D23 92.6 mm to (186.0, 75.0), turned to 180 degrees
- moved D13 89.7 mm to (186.0, 95.0), turned to 180 degrees
- moved D17 87.9 mm to (186.0, 89.5), turned to 180 degrees
- moved D15 87.8 mm to (186.0, 84.0), turned to 180 degrees
- moved D21 87.2 mm to (180.5, 69.5), turned to 180 degrees
- moved D11 87.0 mm to (180.5, 89.5), turned to 180 degrees
- moved D26 84.1 mm to (175.0, 69.5), turned to 180 degrees
- moved U5 84.0 mm to (167.5, 70.0)
- moved D22 83.0 mm to (175.0, 64.0), turned to 180 degrees
- moved D12 82.6 mm to (175.0, 84.0), turned to 180 degrees
- moved D24 82.0 mm to (175.0, 75.0), turned to 180 degrees
- moved R232 81.6 mm to (186.0, 76.5), turned to 180 degrees
- moved D14 78.5 mm to (175.0, 95.0), turned to 180 degrees
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- renumbered R19 to R111, R29 to R112, R15 to R121, R30 to R122, R20 to R131, R31 to R132, R21 to R141, R32 to R142, R16 to R151, R33 to R152, R18 to R161, R34 to R162, R17 to R171, R35 to R172, R12 to R211, R22 to R212, R8 to R221, R23 to R222, R13 to R231, R24 to R232, R14 to R241, R25 to R242, R9 to R251, R26 to R252, R11 to R261, R27 to R262, R10 to R271, R28 to R272
Connections:
- D21 pad 2: Net-(D4-K) -> Net-(D21-K)
- D22 pad 2: Net-(D5-K) -> Net-(D22-K)
- D23 pad 2: Net-(D6-K) -> Net-(D23-K)
- D24 pad 2: Net-(D7-K) -> Net-(D24-K)
- D25 pad 2: Net-(D8-K) -> Net-(D25-K)
- D26 pad 2: Net-(D9-K) -> Net-(D26-K)
- D27 pad 2: Net-(D10-K) -> Net-(D27-K)
- J2 pad MP: unconnected-(J2-PadMP) -> (no net)
- R111 pad 1: Net-(U2-Q6) -> Net-(U2-Q0)
- R121 pad 1: Net-(U2-Q4) -> Net-(U2-Q3)
- R131 pad 1: Net-(U2-Q7) -> Net-(U2-Q3)
- R141 pad 1: Net-(U2-Q7) -> Net-(U2-Q2)
- R151 pad 1: Net-(U2-Q5) -> Net-(U2-Q2)
- R161 pad 1: Net-(U2-Q6) -> Net-(U2-Q1)
- R171 pad 1: Net-(U2-Q5) -> Net-(U2-Q1)
- R211 pad 1: Net-(U2-Q2) -> Net-(U2-Q4)
- R221 pad 1: Net-(U2-Q0) -> Net-(U2-Q7)
- R231 pad 1: Net-(U2-Q3) -> Net-(U2-Q7)
- R241 pad 1: Net-(U2-Q3) -> Net-(U2-Q6)
- R251 pad 1: Net-(U2-Q1) -> Net-(U2-Q6)
- R261 pad 1: Net-(U2-Q2) -> Net-(U2-Q5)
- R271 pad 1: Net-(U2-Q1) -> Net-(U2-Q5)
- U5 pad 10: Net-(D10-K) -> Net-(D24-K)
- U5 pad 11: Net-(D9-K) -> Net-(D23-K)
- U5 pad 12: Net-(D8-K) -> Net-(D21-K)
- U5 pad 13: Net-(D7-K) -> Net-(D26-K)
- U5 pad 14: Net-(D6-K) -> Net-(D27-K)
- U5 pad 15: Net-(D5-K) -> Net-(D25-K)
- U5 pad 16: Net-(D4-K) -> Net-(D22-K)
- U6 pad 10: Net-(D17-K) -> Net-(D14-K)
- U6 pad 11: Net-(D16-K) -> Net-(D13-K)
- U6 pad 12: Net-(D15-K) -> Net-(D11-K)
- U6 pad 13: Net-(D14-K) -> Net-(D16-K)
- U6 pad 14: Net-(D13-K) -> Net-(D17-K)
- U6 pad 15: Net-(D12-K) -> Net-(D15-K)
- U6 pad 16: Net-(D11-K) -> Net-(D12-K)
Routing:
- net 3V3: track 0.00 -> 199.4 mm, vias 0 -> 15
- net /~{RESET}: track 0.00 -> 42.7 mm, vias 0 -> 2
- net GND: track 0.00 -> 36.8 mm, vias 0 -> 44
- net Net-(U2-Q2): track 0.00 -> 35.4 mm, vias 0 -> 2
- net Net-(U2-Q3): track 0.00 -> 30.8 mm, vias 0 -> 2
- net /V_{BAT}: track 0.00 -> 29.7 mm
- net Net-(U2-Q0): track 0.00 -> 28.2 mm
- net /V_{USB-filt}: track 0.00 -> 24.0 mm
- net Net-(U2-Q1): track 0.00 -> 23.4 mm
- net /CLOCK: track 0.00 -> 22.4 mm
- net /DATA: track 0.00 -> 21.5 mm
- net Net-(U2-Q6): track 0.00 -> 20.2 mm, vias 0 -> 2
- net Net-(U2-Q7): track 0.00 -> 19.5 mm, vias 0 -> 2
- net /MOSI: track 0.00 -> 16.3 mm, vias 0 -> 2
- net Net-(D23-K): track 0.00 -> 16.0 mm
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- added copper zone on B.Cu, net GND
- added copper zone on F.Cu, net GND
Other:
- board outline added: 80 x 40 mm
- board text added: "${COMPANY} ${COMMENT1}"
- board text added: "${TITLE}"
- board text added: "Rev: ${REVISION}"
