File: ThreeMan_HW.kicad_sch (KiCad schematic)
At the start: 8 parts, among them J1 USB4135-GF-A, U1 MCP73831T-2ACI/OT

Commit message: Imported updated schematic drawing
Other:
- company: (none) -> Zkylark Electronics

Commit message: Finished initial draft of A1 schematic and imported it to PCB
Parts:
- removed SW?: Off-Mom, Button_Switch_SMD:SW_SPST_PTS645, symbol Switch:PTS645SL43SMTR92_LFS
- added C1, C2: 4u7, Capacitor_SMD:C_0603_HS, symbol Capacitor:C_Generic
- added C3, C4, C5, C6, C7, C8, C9: 100u, Capacitor_SMD:C_0603_HS, symbol Capacitor:C_Generic
- added D1: SMAJ5.0A, Diode_SMD:DO-214AC, symbol Diode_Zener:SMAJ5.0A-13-F
- added D10, D11, D12, D13, D14, D15, D16, D17, D4, D5, D6, D7, D8, D9: Colour, LED_SMD:LED_0603_HS, symbol LED:LED_Generic
- added D2: Red, LED_SMD:LED_0603_HS, symbol LED:LED_Generic
- added D3: Green, LED_SMD:LED_0603_HS, symbol LED:LED_Generic
- added J2: JST-PH-2mm, Connector_JST:JST_PH_S2B-PH-SM4-TB_1x02-1MP_P2.00mm_Horizontal, symbol Connector_JST:S2B-PH-SM4
- added R10, R11, R12, R13, R14, R15, R16, R17, R18, R19, R20, R21, R6, R8, R9: 0R, Resistor_SMD:R_0603_HS, symbol Resistor:R_Generic
- added R22, R23, R24, R25, R26, R27, R28, R29, R30, R31, R32, R33, R34, R35: 120R, Resistor_SMD:R_0603_HS, symbol Resistor:R_Generic
- added R3, R4: R, Resistor_SMD:R_0603_HS, symbol Resistor:R_Generic
- added R5: 2k, Resistor_SMD:R_0603_HS, symbol Resistor:R_Generic
- added R7: 10k, Resistor_SMD:R_0603_HS, symbol Resistor:R_Generic
- added SW1: Off-Mom, Switch_Button_SMD:SW_SPST_PTS645, symbol Switch_Button:PTS645SL43SMTR92_LFS
- added SW2: SW_SPDT_312, Switch_Slide_SMD:CSS-1210TB, symbol Switch_Slide:CSS-1210TB
- added U4: TPS7A20, Package_TO_SOT_SMD:SOT-23-5, symbol Regulator_Linear:TPS7A20
- added U5, U6: ULQ2003D, Package_SO:SOIC-16-N_3.8x9.8mm_P1.27mm, symbol Transistor_Array:ULQ2003D
- J3: renamed from J?; value Conn_TagConnect_TC2030_ICSP -> TC2030_ICSP; Drawing https://github.com/znibb/KiCad-Libraries/blob/main/Datashee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 -> ${DATASHEETS}/Connector/TC2030-IDC-FP-Drawing.pdf
- R1, R2: footprint (none) -> Resistor_SMD:R_0603_HS; Power (none) -> 0.125W
- gave numbers to parts that had none: 2
Connections:
- net GND: now reaches J1.A12 (GND), J1.B12 (GND), R1.2, R2.2
- net GND: now also J3.6 (GND), U1.2 (V_{SS}), U2.13 (~{OE}), U2.8 (GND), U3.4 (GND), C1.2, C2.2, C3.2, C4.2, C5.2, C6.2, C7.2, C8.2, C9.2, D1.2 (A), J2.2 (GND), R4.1, R5.2, SW1.1, U4.2 (GND), U5.8 (E), U6.8 (E)
- net V_{USB}: now reaches J1.A9 (VBUS), J1.B9 (VBUS)
- net V_{USB}: now also R6.1
- net at U1.1 (STAT): now also D2.2 (K), D3.1 (A)
- net V_{BAT}: now reaches U1.3 (V_{BAT})
- net V_{BAT}: now also C2.1, C3.1, J2.1 (V_{BAT}), SW2.3 (C), U4.1 (IN)
- net V_{USB-filt}: now reaches U1.4 (V_{DD})
- net V_{USB-filt}: now also C1.1, C6.1, D1.1 (K), R3.1, R6.2
- net at U1.5 (PROG): now also R5.1
- net at U2.1 (Q1): now also R10.1, R9.1
- net 3V3: now reaches U2.10 (~{MR}), U2.16 (VCC)
- net 3V3: now also J3.2 (VCC), U3.8 (VCC), C5.1, C7.1, C9.1, R22.2, R23.2, R24.2, R25.2, R26.2, R27.2, R28.2, R29.2, R30.2, R31.2, R32.2, R33.2, R34.2, R35.2, R7.1, U4.5 (OUT)
- net CLOCK: now reaches U2.11 (SHCLK)
- net CLOCK: now also U2.12 (STCLK), U3.3 (XTAL2/PB4)
- net DATA: now reaches U2.14 (DATA)
- net DATA: now also U3.2 (XTAL1/PB3)
- net at U2.15 (Q0): now also R8.1
- net at U2.2 (Q2): now also R11.1, R12.1
- net at U2.3 (Q3): now also R13.1, R14.1
- net at U2.4 (Q4): now also R15.1
- net at U2.5 (Q5): now also R16.1, R17.1
- net at U2.6 (Q6): now also R18.1, R19.1
- net at U2.7 (Q7): now also R20.1, R21.1
- net ~{RESET}: now reaches U3.1 (~{RESET}/PB5)
- net ~{RESET}: now also J3.5 (~{RESET}), C8.1, R7.2, SW1.2
- net MOSI: now reaches U3.5 (AREF/PB0)
- net MOSI: now also J3.3 (SCK)
- net MISO: now reaches U3.6 (PB1)
- net MISO: now also J3.1 (MISO)
- net SCK: now reaches U3.7 (PB2)
- net SCK: now also J3.4 (MOSI)
- new net: R20.2, U6.6 (B6)
- new net: R21.2, U6.7 (B7)
- new net: D10.1 (A), R28.1
- new net: D10.2 (K), U5.10 (C7)
- new net: R17.2, U6.3 (B3)
- new net: D14.1 (A), R32.1
- new net: SW2.2 (B), U4.3 (EN)
- new net: D9.1 (A), R27.1
- new net: D9.2 (K), U5.11 (C6)
- new net: D3.2 (K), R4.2
- new net: C4.1, U4.4 (NR)
- new net: D11.1 (A), R29.1
- new net: R8.2, U5.1 (B1)
- new net: D4.1 (A), R22.1
- new net: D4.2 (K), U5.16 (C1)
- new net: D7.1 (A), R25.1
- new net: D12.1 (A), R30.1
- new net: D16.1 (A), R34.1
- new net: D6.1 (A), R24.1
- new net: D5.1 (A), R23.1
- new net: D5.2 (K), U5.15 (C2)
- new net: D15.1 (A), R33.1
- new net: D15.2 (K), U6.12 (C5)
- new net: D13.1 (A), R31.1
- new net: R10.2, U5.3 (B3)
- new net: R18.2, U6.4 (B4)
- new net: D8.1 (A), R26.1
- new net: D8.2 (K), U5.12 (C5)
- new net: R12.2, U5.5 (B5)
- new net: D7.2 (K), U5.13 (C4)
- new net: D16.2 (K), U6.11 (C6)
- new net: D17.1 (A), R35.1
- new net: D2.1 (A), R3.2
- new net: D6.2 (K), U5.14 (C3)
- new net: R9.2, U5.2 (B2)
- new net: R11.2, U5.4 (B4)
- new net: R13.2, U5.6 (B6)
- new net: R14.2, U5.7 (B7)
- new net: D17.2 (K), U6.10 (C7)
- new net: D13.2 (K), U6.14 (C3)
- new net: R15.2, U6.1 (B1)
- new net: R16.2, U6.2 (B2)
- new net: D14.2 (K), U6.13 (C4)
- new net: D12.2 (K), U6.15 (C2)
- new net: D11.2 (K), U6.16 (C1)
- new net: R19.2, U6.5 (B5)
- no-connect marks 1 -> 5
Other:
- moved on the sheet: J1, J3, R1, R2, U1, U2, U3

Commit message: Completed layout
Parts:
- removed SW1: Off-Mom, Switch_Button_SMD:SW_SPST_PTS645, symbol Switch_Button:PTS645SL43SMTR92_LFS
- added H1, H2, H3, H4: M3, MountingHole:MountingHole_3.2mm_M3_Pad, symbol Mechanical:MountingHole_Pad_MP
- added SW1: SW_Push, Switch_Button_SMD:SW_SPST_TS04-66-95-BK-160-SMT, symbol Switch_Button:TS04-66-95-BK-160-SMT
- C1, C2: Tolerance (none) -> 10%
- C3, C4, C5, C6, C7, C8, C9: value 100u -> 100n; Tolerance (none) -> 10%
- D1: DK_PartNo (none) -> SMAJ5.0ALFCT-ND; MPN (none) -> SMAJ5.0A; Manufacturer (none) -> Littelfuse Inc.
- D11, D12, D13, D14, D15, D16, D17: value Colour -> Red
- D21: renamed from D4; value Colour -> Red
- D22: renamed from D5; value Colour -> Red
- D23: renamed from D6; value Colour -> Red
- D24: renamed from D7; value Colour -> Red
- D25: renamed from D8; value Colour -> Red
- D26: renamed from D9; value Colour -> Red
- D27: renamed from D10; value Colour -> Red
- J1: MPN (none) -> USB4135-GF-A
- J2: MPN (none) -> S2B-PH-SM4-TB
- R3, R4: value R -> 590R
- SW2: DK_PartNo (none) -> 563-1091-1-ND; MPN (none) -> CSS-1210TB
- renumbered R19 to R111, R29 to R112, R15 to R121, R30 to R122, R20 to R131, R31 to R132, R21 to R141, R32 to R142, R16 to R151, R33 to R152, R18 to R161, R34 to R162, R17 to R171, R35 to R172, R12 to R211, R22 to R212, R8 to R221, R23 to R222, R13 to R231, R24 to R232, R14 to R241, R25 to R242, R9 to R251, R26 to R252, R11 to R261, R27 to R262, R10 to R271, R28 to R272
Connections:
- net GND: now also SW1.1
- net ~{RESET}: now also SW1.2
- net at D27.2 (K): now also U5.14 (C3); no longer U5.10 (C7)
- net at D26.2 (K): now also U5.13 (C4); no longer U5.11 (C6)
- net at R221.1: now also R231.1, U2.7 (Q7); no longer U2.15 (Q0)
- net at D21.2 (K): now also U5.12 (C5); no longer U5.16 (C1)
- net at D22.2 (K): now also U5.16 (C1); no longer U5.15 (C2)
- net at D15.2 (K): now also U6.15 (C2); no longer U6.12 (C5)
- net at D25.2 (K): now also U5.15 (C2); no longer U5.12 (C5)
- net at R121.1: now also R131.1, U2.3 (Q3); no longer U2.4 (Q4)
- net at D24.2 (K): now also U5.10 (C7); no longer U5.13 (C4)
- net at D16.2 (K): now also U6.13 (C4); no longer U6.11 (C6)
- net at D23.2 (K): now also U5.11 (C6); no longer U5.14 (C3)
- net at D17.2 (K): now also U6.14 (C3); no longer U6.10 (C7)
- net at D13.2 (K): now also U6.11 (C6); no longer U6.14 (C3)
- net at D14.2 (K): now also U6.10 (C7); no longer U6.13 (C4)
- net at D12.2 (K): now also U6.16 (C1); no longer U6.15 (C2)
- net at D11.2 (K): now also U6.12 (C5); no longer U6.16 (C1)
- new net: R141.1, R151.1, U2.2 (Q2)
- new net: R161.1, R171.1, U2.1 (Q1)
- new net: R261.1, R271.1, U2.5 (Q5)
- new net: R111.1, U2.15 (Q0)
- new net: R211.1, U2.4 (Q4)
- new net: R241.1, R251.1, U2.6 (Q6)
- no-connect marks 5 -> 9
Other:
- title: Three Man -> ThreeMan
- moved on the sheet: C1, C2, C6, D1, D11, D12, D13, D14, D15, D16, D17, D21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
